File: power.kicad_sch (KiCad schematic)
At the start: 0 parts

Commit message: added power management unit
Parts:
- added IC1: TPS63070RNMR, TPS630701RNMR, symbol TPS63070RNMR:TPS63070RNMR
Changed lines of the file:
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@@
 	(generator_version "9.0")
 	(paper "A4")
+	(symbol
+		(lib_id "TPS63070RNMR:TPS63070RNMR")
+		(at 134.62 90.17 0)
+		(unit 1)
+		(exclude_from_sim no)
+		(in_bom yes)
+		(on_board yes)
+		(dnp no)
+		(fields_autoplaced yes)
+		(property "Reference" "IC1"
+			(at 151.13 82.55 0)
+			(effects
+				(font
+					(size 1.27 1.27)
+				)
+			)
+		)
+		(property "Value" "TPS63070RNMR"
+			(at 151.13 85.09 0)
+			(effects
+				(font
+					(size 1.27 1.27)
+				)
+			)
+		)
+		(property "Footprint" "TPS630701RNMR"
+			(at 163.83 185.09 0)
+			(effects
+				(font
+					(size 1.27 1.27)
+				)
+				(justify left top)
+				(hide yes)
+			)
+		)
+		(property "Datasheet" "http://www.ti.com/lit/gpn/tps63070"
+			(at 163.83 285.09 0)
+			(effects
+				(font
+					(size 1.27 1.27)
+				)
+				(justify left top)
+				(hide yes)
+			)
+		)
+		(property "Description" "Wide Input Voltage (2V-16V) Buck-Boost Converter"
+			(at 134.62 90.17 0)
+			(effects
+				(font
+					(size 1.27 1.27)
+				)
+				(hide yes)
+			)
+		)
+		(property "Height" ""
+			(at 163.83 485.09 0)
+			(effects
+				(font
+					(size 1.27 1.27)
+				)
+				(justify left top)
+				(hide yes)
+			)
+		)
+		(property "Mouser Part Number" "595-TPS63070RNMR"
+			(at 163.83 585.09 0)
+			(effects
+				(font
+					(size 1.27 1.27)
+				)
+				(justify left top)
+				(hide yes)
+			)
+		)
+		(property "Mouser Price/Stock" "https://www.mouser.co.uk/ProductDetail/Texas-Instruments/TPS63070RNMR?qs=LuYMPh7GGMS51GHntBDRnQ%3D%3D"
+			(at 163.83 685.09 0)
+			(effects
+				(font
+					(size 1.27 1.27)
+				)
+				(justify left top)
+				(hide yes)
+			)
+		)
+		(property "Manufacturer_Name" "Texas Instruments"
+			(at 163.83 785.09 0)
+			(effects
+				(font
+					(size 1.27 1.27)
+				)
+				(justify left top)
+				(hide yes)
+			)
+		)
+		(property "Manufacturer_Part_Number" "TPS63070RNMR"
+			(at 163.83 885.09 0)
+			(effects
+				(font
+					(size 1.27 1.27)
+				)
+				(justify left top)
+				(hide yes)
+			)
+		)
+		(pin "1"
+		)
+		(pin "7"
+		)
+		(pin "8"
+		)
+		(pin "9"
+		)
+		(pin "10"
+		)
+		(pin "11"
+		)
+		(pin "12"
+		)
+		(pin "13"
+		)
+		(pin "14"
+		)
+		(pin "15"
+		)
+		(pin "4"
+		)
+		(pin "2"
+		)
+		(pin "3"
+		)
+		(pin "5"
+		)
+		(pin "6"
+		)
+		(instances
+			(project ""
+				(path "/8edf12b2-d2f1-4d92-9f83-70002c2ec599"
+					(reference "IC1")
+					(unit 1)
+				)
+			)
+		)
+	)
+	(sheet_instances
+		(path "/"
+			(page "1")
+		)
+	)
+	(embedded_fonts no)
 )

Commit message: Finish voltage regulator schematic
Parts:
- added C23: 100n, symbol Device:C
- added C24, C28, C29, C30: 10u, symbol Device:C
- added C25, C26, C27: 22u, symbol Device:C
- added L8: 1.5u, symbol Device:L
- added R2: 100k, symbol Device:R_US
- added R3: 10k, symbol Device:R_US
- added R4: 470k, symbol Device:R_US
- added R5: 150k, symbol Device:R_US
Connections:
- net at IC1.1 (PS/S): now also IC1.14 (EN), R3.1
- net GND: now reaches IC1.10 (PGND)
- net GND: now also IC1.15 (VSEL), IC1.4 (GND), IC1.6 (FB2), C23.1, C24.2, C25.2, C26.2, C27.2, C28.2, C29.2, C30.2, R5.2
- net at IC1.11 (L1): now also L8.2
- net V_BATT: now reaches IC1.13 (VIN_2)
- net V_BATT: now also C28.1, C29.1, C30.1, R3.2
- net at IC1.2 (PG): now also R2.1
- net at IC1.3 (VAUX): now also C23.2
- net at IC1.5 (FB): now also R4.1
- net 3V3: now reaches IC1.8 (VOUT_2)
- net 3V3: now also C24.1, C25.1, C26.1, C27.1, R2.2, R4.2, R5.1
- net at IC1.9 (L2): now also L8.1
- no-connect marks 0 -> 2
